Commit message: Add Gazebo colors

File: linorobot2_description/urdf/robots/nexusurdf.xacro (robot description, xacro)
@@ -52,17 +52,4 @@
     </inertial>
   </link>
-  <gazebo reference="base_link">
-    <material>Gazebo/Yellow</material>
-  </gazebo>
-    <!-- <gazebo reference="base_link">
-      <visual>
-        <material>
-          <ambient>0.8392 0.6314 0.0 1.0</ambient>
-          <diffuse>0.8392 0.6314 0.0 1.0</diffuse>
-          <specular>0.99 0.99 0.99 1.0</specular>
-          <emissive>0.0 0.0 0.0 0.0</emissive>
-        </material>
-      </visual>
-    </gazebo> -->
   <joint name="upper_left_wheel_shaft_joint" type="fixed">
     <origin xyz="0.150 0.108 0.0" rpy="0 0 0" />
@@ -93,7 +80,4 @@
     </inertial>
   </link>
- <gazebo reference="upper_left_wheel_shaft">
-    <material>Gazebo/Black</material>
-  </gazebo>
   <joint name="lower_left_wheel_shaft_joint" type="fixed">
     <origin xyz="-0.150 0.108 0.0" rpy="0 0 0" />
@@ -210,10 +194,4 @@
     </inertial>
   </link>
-  <!-- Wheel friction to zero, as movement is handled by applying forces at the body level. -->
-  <gazebo reference="upper_left_wheel">
-    <material>Gazebo/Grey</material>
-    <mu1>0.0</mu1>
-    <mu2>0.0</mu2>
-  </gazebo>
   <joint name="lower_left_wheel_joint" type="continuous">
     <origin xyz="0 0.042 0" rpy="0 0 0" />
@@ -362,48 +340,4 @@
     </visual>
   </link>
-  <!-- <xacro:base
-    length="${base_length}"
-    width="${base_width}"
-    height="${base_height}"
-    mass="${base_mass}"
-    wheel_radius="${wheel_radius}"
-    wheel_pos_z="${wheel_pos_z}"
-/>
-  <xacro:mecanum_wheel
-    side="front_left"
-    radius="${wheel_radius}"
-    width="${wheel_width}"
-    pos_x="${wheel_pos_x}"
-    pos_y="${wheel_pos_y}"
-    pos_z="${wheel_pos_z}"
-    mass="${wheel_mass}"
-  />
-  <xacro:mecanum_wheel
-    side="front_right"
-    radius="${wheel_radius}"
-    width="${wheel_width}"
-    pos_x="${wheel_pos_x}"
-    pos_y="${-wheel_pos_y}"
-    pos_z="${wheel_pos_z}"
-    mass="${wheel_mass}"
-  />
-  <xacro:mecanum_wheel
-    side="rear_left"
-    radius="${wheel_radius}"
-    width="${wheel_width}"
-    pos_x="${-wheel_pos_x}"
-    pos_y="${wheel_pos_y}"
-    pos_z="${wheel_pos_z}"
-    mass="${wheel_mass}"
-  />
-  <xacro:mecanum_wheel
-    side="rear_right"
-    radius="${wheel_radius}"
-    width="${wheel_width}"
-    pos_x="${-wheel_pos_x}"
-    pos_y="${-wheel_pos_y}"
-    pos_z="${wheel_pos_z}"
-    mass="${wheel_mass}"
-  /> -->
   <xacro:imu/>
   <xacro:generic_laser>
@@ -414,3 +348,55 @@
   </xacro:depth_sensor>
   <xacro:omni_drive_controller/>
+   <gazebo reference="base_footprint">
+    <material>Gazebo/Yellow</material>
+    <gravity>true</gravity>
+  </gazebo>
+  <gazebo reference="base_link">
+    <material>Gazebo/Yellow</material>
+  </gazebo>
+  <gazebo reference="left_sensor">
+    <material>Gazebo/Black</material>
+  </gazebo>
+   <gazebo reference="front_sensor">
+    <material>Gazebo/Black</material>
+  </gazebo>
+   <gazebo reference="right_sensor">
+    <material>Gazebo/Black</material>
+  </gazebo>
+   <gazebo reference="rear_sensor">
+    <material>Gazebo/Black</material>
+  </gazebo>
+  <gazebo reference="upper_left_wheel_shaft">
+    <material>Gazebo/Black</material>
+  </gazebo>
+  <gazebo reference="lower_left_wheel_shaft">
+    <material>Gazebo/Black</material>
+  </gazebo>
+  <gazebo reference="upper_right_wheel_shaft">
+    <material>Gazebo/Black</material>
+  </gazebo>
+  <gazebo reference="lower_right_wheel_shaft">
+    <material>Gazebo/Black</material>
+  </gazebo>
+  <!-- Wheel friction to zero, as movement is handled by applying forces at the body level. -->
+  <gazebo reference="upper_left_wheel">
+    <material>Gazebo/Grey</material>
+    <mu1>0.0</mu1>
+    <mu2>0.0</mu2>
+  </gazebo>
+  <gazebo reference="lower_left_wheel">
+    <material>Gazebo/Grey</material>
+    <mu1>0.0</mu1>
+    <mu2>0.0</mu2>
+  </gazebo>
+  <gazebo reference="upper_right_wheel">
+    <material>Gazebo/Grey</material>
+    <mu1>0.0</mu1>
+    <mu2>0.0</mu2>
+  </gazebo>
+  <gazebo reference="lower_right_wheel">
+    <material>Gazebo/Grey</material>
+    <mu1>0.0</mu1>
+    <mu2>0.0</mu2>
+  </gazebo>
 </robot>

Commit message: Adjust Rviz and Gazeco colors

File: linorobot2_description/urdf/robots/nexusurdf.xacro (robot description, xacro)
@@ -8,9 +8,11 @@
   <xacro:include filename="$(find linorobot2_description)/urdf/sensors/depth_sensor.urdf.xacro" />
   <xacro:include filename="$(find linorobot2_description)/urdf/controllers/omni_drive.urdf.xacro" />
+<!-- robcomw: -->
+  <xacro:include filename="$(find linorobot2_description)/urdf/common_constants.xacro" />
 <!-- Using `package://` in URDF with ROS2 -->
 <!-- https://answers.ros.org/question/370075/using-package-in-urdf-with-ros2/ -->
  <!-- place meshes in install/linorobot2_description/share/linorobot2_description/mech -->
 <!-- /ros2_ws/src/linorobot2/linorobot2_description/urdf/robots -->
-  <xacro:property name="PI" value="3.1415926535897931" />
+  <!-- <xacro:property name="PI" value="3.1415926535897931" /> -->
   <xacro:property name="wheel_radius" value="0.050" />
   <xacro:property name="wheel_width" value="0.0505" />

File: linorobot2_description/urdf/sensors/depth_sensor.urdf.xacro (robot description, xacro)
@@ -1,15 +1,34 @@
 <robot xmlns:xacro="http://ros.org/wiki/xacro">
   <xacro:property name="M_PI" value="3.1415926535897931" />
+  <!-- robcomw: -->
+  <xacro:include filename="$(find linorobot2_description)/urdf/common_constants.xacro" />
+  <!-- <material name="yellow"><color rgba="0.8 0.8 0.0 1.0" /></material>
+  <material name="black"><color rgba="0.15 0.15 0.15 1.0" /></material>
+  <material name="dark_grey"><color rgba="0.2 0.2 0.2 1.0" /></material>
+  <material name="light_grey"><color rgba="0.4 0.4 0.4 1.0" /></material> -->
   <xacro:macro name="depth_sensor" params="*origin">
     <link name="camera_link">
       <visual>
-        <origin xyz="0 0 0" rpy="0 0 0"/>
+        <!-- <origin xyz="0 0 0" rpy="0 0 0"/> -->
+        <origin xyz="0 0 -0" rpy="${ROTATE_90_DEGREES} 0 ${ROTATE_90_DEGREES}"/>
         <geometry>
-          <box size="0.030 0.124 0.030"/>
+          <!-- <box size="0.030 0.124 0.030"/> -->
           <!-- <mesh filename="" scale="0.001 0.001 0.001"/> -->
+          <mesh filename="file://$(find linorobot2_description)/meshes/intel_realsense_d435.STL" scale="0.001 0.001 0.001"/>
         </geometry>
-        <material name="red">
+        <!-- <material name="light_grey" /> -->
+        <material name="silver">
+          <color rgba="0.75 0.75 0.75 1.0"/> <!-- Adjust the rgba values as needed -->
+        </material>
+        <!-- <material name="light_grey">
+          <color rgba="0.4 0.4 0.4 1.0" />
+        </material> -->
+        <!-- <material>Gazebo/DarkGrey</material> -->
+        <!-- <material name="red">
           <color rgba="0.416 0.051 0.047 1.0"/>
-        </material>
+        </material> -->
+        <!-- <material name="green">
+            <color rgba="0.003 0.639 0.223 1.0"/>
+        </material> -->
       </visual>
       <collision>
@@ -27,4 +46,5 @@
       </inertial>
     </link>
+<!--
     <gazebo reference="camera_link">
       <visual>
@@ -36,5 +56,92 @@
         </material>
       </visual>
-    </gazebo>rgb(213,28,40)
+    </gazebo>rgb(213,28,40) -->
+    <!--silver color-->
+    <!-- <gazebo reference="camera_link">
+      <visual>
+        <material>
+          <ambient>0.192 0.192 0.192 1.0</ambient>
+          <diffuse>0.507 0.507 0.507 1.0</diffuse>
+          <specular>0.508 0.508 0.508 1.0</specular>
+          <emissive>0.0 0.0 0.0 0.0</emissive>
+        </material>
+      </visual>
+    </gazebo> -->
+            <!-- Adjusted RGBA values for glossy silver -->
+    <!-- <gazebo reference="camera_link">
+        <visual>
+            <material>
+                <ambient>0.6 0.6 0.6 1.0</ambient>
+                <diffuse>0.8 0.8 0.8 1.0</diffuse>
+                <specular>0.9 0.9 0.9 1.0</specular>
+                <emissive>0.0 0.0 0.0 0.0</emissive>
+            </material>
+        </visual>
+    </gazebo> -->
+    <!-- <gazebo reference="camera_link">
+        <visual>
+            <material>
+                <ambient>0.8 0.8 0.8 1.0</ambient>
+                <diffuse>0.9 0.9 0.9 1.0</diffuse>
+                <specular>1.0 1.0 1.0 1.0</specular>
+                <emissive>0.0 0.0 0.0 0.0</emissive>
+            </material>
+        </visual>
+    </gazebo> -->
+    <!-- <gazebo reference="camera_link">
+        <visual>
+            <material>
+                <ambient>0.9 0.9 0.9 1.0</ambient>
+                <diffuse>0.95 0.95 0.95 1.0</diffuse>
+                <specular>1.0 1.0 1.0 1.0</specular>
+                <emissive>0.0 0.0 0.0 0.0</emissive>
+            </material>
+        </visual>
+    </gazebo> -->
+    <!-- <gazebo reference="camera_link">
+        <visual>
+            <material>
+                <ambient>0.8 0.8 0.8 1.0</ambient>
+                <diffuse>0.9 0.9 0.9 1.0</diffuse>
+                <specular>1.0 1.0 1.0 1.0</specular>
+                <emissive>0.05 0.05 0.05 0.0</emissive>
+            </material>
+        </visual>
+    </gazebo> -->
+    <!-- <gazebo reference="camera_link">
+        <visual>
+            <material name="light_grey">
+                <color rgba="0.4 0.4 0.4 1.0"/>
+            </material>
+        </visual>
+    </gazebo> -->
+    <!-- <gazebo reference="camera_link">
+        <visual>
+            <material name="dark_grey">
+                <color rgba="0.3 0.3 0.3 1.0"/>
+            </material>
+        </visual>
+    </gazebo> -->
+      <!-- LIGHTER DARK GREY  -->
+    <!-- <gazebo reference="camera_link">
+        <visual>
+          <material>
+            <ambient>0.6 0.6 0.6 1.0</ambient>
+            <diffuse>0.8 0.8 0.8 1.0</diffuse>
+            <specular>0.4 0.4 0.4 1.0</specular>
+            <emissive>0.0 0.0 0.0 0.0</emissive>
+          </material>
+        </visual>
+    </gazebo> -->
+    <gazebo reference="camera_link">
+        <visual>
+            <material>
+                <ambient>0.8 0.8 0.8 1.0</ambient>
+                <diffuse>0.9 0.9 0.9 1.0</diffuse>
+                <specular>1.0 1.0 1.0 1.0</specular>
+                <emissive>0.0 0.0 0.0 0.0</emissive>
+            </material>
+        </visual>
+    </gazebo>
     <joint name="camera_to_base_link" type="fixed">
       <parent link="base_link"/>

File: linorobot2_description/urdf/sensors/laser.urdf.xacro (robot description, xacro)
@@ -1,15 +1,31 @@
 <robot xmlns:xacro="http://ros.org/wiki/xacro">
-  <xacro:property name="M_PI" value="3.1415926535897931" />
+  <!-- robcomw: -->
+  <xacro:include filename="$(find linorobot2_description)/urdf/common_constants.xacro" />
+  <!-- <material name="yellow"><color rgba="0.8 0.8 0.0 1.0" /></material>
+  <material name="black"><color rgba="0.15 0.15 0.15 1.0" /></material>
+  <material name="dark_grey"><color rgba="0.2 0.2 0.2 1.0" /></material>
+  <material name="light_grey"><color rgba="0.4 0.4 0.4 1.0" /></material> -->
   <xacro:macro name="laser" params="*origin update_rate ray_count min_angle max_angle min_range max_range frame_id topic_name">
     <link name="${frame_id}">
       <visual>
         <!-- <origin xyz="0 0 -0.025" rpy="0 0 0"/> -->
-        <origin xyz="0 0 0.016" rpy="0 0 0"/>
+        <!-- <origin xyz="0 0 0.016" rpy="0 0 0"/> -->
+        <!-- <origin xyz="0 0.06067 -0.009" rpy="${ROTATE_90_DEGREES} 0 ${ROTATE_90_DEGREES}"/>  -->
+        <!-- <origin xyz="0 0.0836 -0.09" rpy="${ROTATE_90_DEGREES} 0 ${ROTATE_90_DEGREES}"/> -->
+        <!-- X OK, Y ON THE PLATE -->
+        <!-- <origin xyz="0 0.0836 -0.019" rpy="${ROTATE_90_DEGREES} 0 ${ROTATE_90_DEGREES}"/>  -->
+        <origin xyz="0 0.0836 -0.019" rpy="${ROTATE_90_DEGREES} 0 ${ROTATE_90_DEGREES}"/>
         <geometry>
           <!-- <cylinder radius="0.0375" length="0.05"/> -->
-          <cylinder radius="0.038" length="0.041"/>
+          <!-- <cylinder radius="0.038" length="0.041"/> -->
+          <mesh filename="file://$(find linorobot2_description)/meshes/rp_lidar_a3.STL" scale="0.001 0.001 0.001"/>
         </geometry>
-        <material name="green">
+        <!-- <material name="green">
             <color rgba="0.003 0.639 0.223 1.0"/>
+        </material> -->
+        <!-- <material name="black" /> -->
+        <!-- <material name="dark_grey"><color rgba="0.2 0.2 0.2 1.0" /></material>         -->
+        <material name="light_dark_gray">
+            <color rgba="0.3 0.3 0.3 1.0"/> <!-- Adjust the rgba values as needed -->
         </material>
       </visual>
@@ -29,5 +45,8 @@
       </inertial>
     </link>
-    <gazebo reference="${frame_id}">
+    <!-- <gazebo reference="c${frame_id}">
+      <material>Gazebo/DarkGrey</material>
+    </gazebo> -->
+    <!-- <gazebo reference="${frame_id}">
       <visual>
         <material>
@@ -38,4 +57,37 @@
         </material>
       </visual>
+    </gazebo> -->
+    <!-- light dark grey  -->
+    <!-- <gazebo reference="${frame_id}">
+        <visual>
+            <material>
+                <ambient>0.2 0.2 0.2 1.0</ambient>
+                <diffuse>0.4 0.4 0.4 1.0</diffuse>
+                <specular>0.1 0.1 0.1 1.0</specular>
+                <emissive>0.0 0.0 0.0 0.0</emissive>
+            </material>
+        </visual>
+    </gazebo> -->
+      <!-- LIGHTER DARK GREY  -->
+    <!-- <gazebo reference="${frame_id}">
+        <visual>
+            <material>
+                <ambient>0.4 0.4 0.4 1.0</ambient>
+                <diffuse>0.6 0.6 0.6 1.0</diffuse>
+                <specular>0.2 0.2 0.2 1.0</specular>
+                <emissive>0.0 0.0 0.0 0.0</emissive>
+            </material>
+        </visual>
+    </gazebo> -->
+      <!-- TOO LIGHT DARK GREY  -->
+    <gazebo reference="${frame_id}">
+        <visual>
+            <material>
+                <ambient>0.6 0.6 0.6 1.0</ambient>
+                <diffuse>0.8 0.8 0.8 1.0</diffuse>
+                <specular>0.4 0.4 0.4 1.0</specular>
+                <emissive>0.0 0.0 0.0 0.0</emissive>
+            </material>
+        </visual>
     </gazebo>
     <joint name="${frame_id}_to_base_link" type="fixed">
